File: Solder_Panel_Idea1.kicad_sch (KiCad schematic)
At the start: 27 parts, among them SW1 SW_Push_Dual_x2, SW2 SW_Push_Dual_x2, SW3 SW_Push_Dual_x2, SW4 SW_Push_Dual_x2, SW5 SW_Push_Dual_x2, SW6 SW_Push_Dual_x2, SW7 SW_Push_Dual_x2, U1 SA555P

Commit message: Yup
Parts:
- C1, C2: footprint Capacitor_SMD:C_1812_4532Metric_Pad1.57x3.40mm_HandSolder -> Capacitor_THT:C_Disc_D7.5mm_W2.5mm_P5.00mm
- C3: footprint Capacitor_THT:CP_Radial_D10.0mm_P5.00mm -> Capacitor_THT:C_Radial_D5.0mm_H7.0mm_P2.00mm
- R1, R10, R11, R12, R13, R14, R2, R3, R4, R5, R6, R7, R8, R9: footprint (none) -> Resistor_THT:R_Axial_DIN0411_L9.9mm_D3.6mm_P15.24mm_Horizontal
Changed lines of the file:
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@@
 			)
 		)
-		(property "Footprint" ""
+		(property "Footprint" "Resistor_THT:R_Axial_DIN0411_L9.9mm_D3.6mm_P15.24mm_Horizontal"
 			(at 139.192 76.2 90)
 			(effects
@@
 			)
 		)
-		(property "Footprint" ""
+		(property "Footprint" "Resistor_THT:R_Axial_DIN0411_L9.9mm_D3.6mm_P15.24mm_Horizontal"
 			(at 250.952 27.94 90)
 			(effects
@@
 			)
 		)
-		(property "Footprint" ""
+		(property "Footprint" "Resistor_THT:R_Axial_DIN0411_L9.9mm_D3.6mm_P15.24mm_Horizontal"
 			(at 160.782 27.94 90)
 			(effects
@@
 			)
 		)
-		(property "Footprint" ""
+		(property "Footprint" "Resistor_THT:R_Axial_DIN0411_L9.9mm_D3.6mm_P15.24mm_Horizontal"
 			(at 228.092 27.94 90)
 			(effects
@@
 			)
 		)
-		(property "Footprint" ""
+		(property "Footprint" "Resistor_THT:R_Axial_DIN0411_L9.9mm_D3.6mm_P15.24mm_Horizontal"
 			(at 139.192 27.94 90)
 			(effects
@@
 			)
 		)
-		(property "Footprint" "Capacitor_SMD:C_1812_4532Metric_Pad1.57x3.40mm_HandSolder"
+		(property "Footprint" "Capacitor_THT:C_Disc_D7.5mm_W2.5mm_P5.00mm"
 			(at 53.0352 72.39 0)
 			(effects
@@
 			)
 		)
-		(property "Footprint" ""
+		(property "Footprint" "Resistor_THT:R_Axial_DIN0411_L9.9mm_D3.6mm_P15.24mm_Horizontal"
 			(at 182.372 76.2 90)
 			(effects
@@
 			)
 		)
-		(property "Footprint" ""
+		(property "Footprint" "Resistor_THT:R_Axial_DIN0411_L9.9mm_D3.6mm_P15.24mm_Horizontal"
 			(at 205.232 27.94 90)
 			(effects
@@
 			)
 		)
-		(property "Footprint" ""
+		(property "Footprint" "Resistor_THT:R_Axial_DIN0411_L9.9mm_D3.6mm_P15.24mm_Horizontal"
 			(at 116.332 27.94 90)
 			(effects
@@
 			)
 		)
-		(property "Footprint" ""
+		(property "Footprint" "Resistor_THT:R_Axial_DIN0411_L9.9mm_D3.6mm_P15.24mm_Horizontal"
 			(at 116.332 76.2 90)
 			(effects
@@
 			)
 		)
-		(property "Footprint" ""
+		(property "Footprint" "Resistor_THT:R_Axial_DIN0411_L9.9mm_D3.6mm_P15.24mm_Horizontal"
 			(at 228.092 76.2 90)
 			(effects
@@
 			)
 		)
-		(property "Footprint" ""
+		(property "Footprint" "Resistor_THT:R_Axial_DIN0411_L9.9mm_D3.6mm_P15.24mm_Horizontal"
 			(at 160.782 76.2 90)
 			(effects
@@
 			)
 		)
-		(property "Footprint" "Capacitor_THT:CP_Radial_D10.0mm_P5.00mm"
+		(property "Footprint" "Capacitor_THT:C_Radial_D5.0mm_H7.0mm_P2.00mm"
 			(at 100.0252 50.8 0)
 			(effects
@@
 			)
 		)
-		(property "Footprint" ""
+		(property "Footprint" "Resistor_THT:R_Axial_DIN0411_L9.9mm_D3.6mm_P15.24mm_Horizontal"
 			(at 205.232 76.2 90)
 			(effects
@@
 			)
 		)
-		(property "Footprint" ""
+		(property "Footprint" "Resistor_THT:R_Axial_DIN0411_L9.9mm_D3.6mm_P15.24mm_Horizontal"
 			(at 250.952 76.2 90)
 			(effects
@@
 			)
 		)
-		(property "Footprint" ""
+		(property "Footprint" "Resistor_THT:R_Axial_DIN0411_L9.9mm_D3.6mm_P15.24mm_Horizontal"
 			(at 182.372 27.94 90)
 			(effects
@@
 			)
 		)
-		(property "Footprint" "Capacitor_SMD:C_1812_4532Metric_Pad1.57x3.40mm_HandSolder"
+		(property "Footprint" "Capacitor_THT:C_Disc_D7.5mm_W2.5mm_P5.00mm"
 			(at 119.0752 91.44 0)
 			(effects

Commit message: hopefully correcting Git
Parts:
- removed SW1, SW2, SW3, SW4, SW5, SW6, SW7: SW_Push_Dual_x2, symbol Switch:SW_Push_Dual_x2
- added S1, S2, S3, S4, S5, S6, S7: TL2201EEYA, TL2201EEYA:SW_TL2201EEYA, symbol TL2201EEYA:TL2201EEYA
- added SW1: SW_SPDT_1825232-1, Swadge-Parts:1825232-1, symbol Swadge_Parts:SW_SPDT_1825232-1
- renumbered C3 to C1, C1 to C2, C2 to C3, R6 to R10, R8 to R11, R10 to R12, R12 to R13, R3 to R2, R5 to R3, R7 to R4, R9 to R5, R11 to R6, R13 to R7, R2 to R8, R4 to R9
Connections:
- net at R1.1, R2.1, R3.1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: now also SW1.3 (C); no longer BT1.P
- net at U1.7 (DIS): now also S1.3, S1.5, S2.3, S2.5, S3.3, S3.5, S4.3, S4.5, S5.3, S5.5, S6.3, S6.5, S7.3, S7.5
- net at R13.1: now also S6.6
- net at R11.1: now also S4.6
- net at R4.2: now also S4.2
- net at R9.1: now also S2.6
- net at R14.1: now also S7.6
- net at R3.2: now also S3.2
- net at R8.1: now also S1.6
- net at R7.2: now also S7.2
- net at R6.2: now also S6.2
- net at R2.2: now also S2.2
- net at R5.2: now also S5.2
- net at R1.2: now also S1.2
- net at R10.1: now also S3.6
- net at R12.1: now also S5.6
- new net: BT1.P, SW1.2 (B)
- no-connect marks 0 -> 17
Other:
- moved on the sheet: BT1, BZ1, C1, C2, C3, R1, R10, R11, R12, R13, R14, R2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
